File: Hardware/base_node/base_node.kicad_sch (KiCad schematic)
At the start: 29 parts, among them J1 IO Interface, J2 RS-422 Connector, J3 Expantion Connector, J4 I2C, J5 24vdc, J6 Encoder 1, J7 Encoder 2, SW1 SW_DIP_x08, U1 CH32X033F8P6, U2 MAX491E, U3 74HC165, U4 MP1584EN_Module

Commit message: docs: establish hierarchical documentation structure and subsystem guides
- Created root navigation hub README.md linking architecture, subsystems, and components
- Added Hardware Subsystem README (bus topology, 24V power rail, RS-422, SM712 protection, BOM)
- Created Base Node README with pinouts (Dev vs Prod), 3D production renders, and manufacturing specs
- Created Gateway Node README with dual-transceiver room segmentation, EEPROM routing, and dev board
- Created Fan Controller Node README with ZCD optocoupler, isolated gate drive, and anti-stall logic
- Created Expanders README with SMD breakout adapter specs and layout previews
- Created Firmware & Protocol Specification README covering 32-bit addressing, packet formats, and dual-slot OTA
- Synchronized KiCad hardware assets, manufacturing plots, and component libraries
Parts:
- removed D2: LED_RGAB, HomeBus:Crystal_SMD_0603-4Pin_6.0x3.5mm_HandSoldering, symbol HomeBus:LED_RGAB
- removed R2, R3: 330Ω, HomeBus:R_0805_2012Metric, symbol HomeBus:R_Small
- added C7: 100nF, HomeBus:C_0603_1608Metric, symbol HomeBus:C_Small
- added D2: WS2812B, HomeBus:XINGLIGHT-XL-1010RGBC-WS2812B, symbol HomeBus:WS2812B
- added D4: SMBJ26A, Diode_SMD:D_SMB, symbol Device:D_TVS
- R1, R4: footprint HomeBus:R_0805_2012Metric -> Resistor_SMD:R_0603_1608Metric
Connections:
- net +5V: now also C7.2, D2.1 (VDD)
- net GND: now also C7.1, D2.3 (VSS), D4.1 (A1)
- net at J1.2 (Pin_2), J6.2 (Pin_2), RN2.2 (R1): now also J3.14 (Pin_14), U1.3 (PB1/A9); no longer J3.8 (Pin_8), U1.20 (PA5)
- net at J3.19 (Pin_19), U1.8 (PC18/SWDIO): now also J1.6 (Pin_6), J7.3 (Pin_3), RN2.6 (R5); no longer J1.8 (Pin_8), RN2.8 (R7)
- net at J3.20 (Pin_20), U1.18 (PC19/SWCLK): now also J1.7 (Pin_7), RN2.7 (R6); no longer J1.9 (Pin_9), RN2.9 (R8)
- net at J3.11 (Pin_11), U1.10 (PA9): now also J1.8 (Pin_8), RN2.8 (R7); no longer R1.1
- net SDA: now reaches J3.13 (Pin_13), U1.11 (PA11/RX1/SDA)
- net SDA: now also J4.3 (Pin_3), R7.2
- net SCL: now reaches J3.12 (Pin_12), U1.12 (PA10/TX1/SCK)
- net SCL: now also J4.4 (Pin_4), R8.2
- net at R1.2: now also D2.4 (DIN)
- net +24vdc renamed +24V
- net +24V: now also D4.2 (A2)
- new net: J1.9 (Pin_9), J3.8 (Pin_8), RN2.9 (R8), U1.20 (PA5)
- new net: J3.17 (Pin_17), U1.5 (PC16), U3.9 (Q7)
- new net: J3.18 (Pin_18), R1.1, U1.6 (PC17)
- no-connect marks 1 -> 2
Other:
- moved on the sheet: R1
