File: Hardware/base_node/base_node_clad_v2.kicad_pcb (KiCad board)
At the start: 2 copper layers, 265 x 165.3 mm, 120 parts, among them J1 IO Interface, J2 RS-422 Connector, J3 Expantion Connector, J4 I2C, J5 Programming Header, J6 Encoder 1, J7 Encoder 2, J8 24vdc, SW1 SW_DIP_x08, U1 CH32X033F8P6, U2 MAX491E, U3 74HC165, U4 MP1584EN_Module

Commit message: docs: establish hierarchical documentation structure and subsystem guides
- Created root navigation hub README.md linking architecture, subsystems, and components
- Added Hardware Subsystem README (bus topology, 24V power rail, RS-422, SM712 protection, BOM)
- Created Base Node README with pinouts (Dev vs Prod), 3D production renders, and manufacturing specs
- Created Gateway Node README with dual-transceiver room segmentation, EEPROM routing, and dev board
- Created Fan Controller Node README with ZCD optocoupler, isolated gate drive, and anti-stall logic
- Created Expanders README with SMD breakout adapter specs and layout previews
- Created Firmware & Protocol Specification README covering 32-bit addressing, packet formats, and dual-slot OTA
- Synchronized KiCad hardware assets, manufacturing plots, and component libraries
Parts:
- removed the C1 at (251.8, 160.9)
- removed the C1 at (116.8, 160.9)
- removed the C1 at (251.8, 75.5)
- removed the C2 at (250.3, 159.4)
- removed the C2 at (115.4, 159.4)
- removed the C2 at (250.4, 74.0)
- removed the C3 at (56.4, 153.8)
- removed the C3 at (191.3, 68.5)
- removed the C3 at (191.3, 153.8)
- removed the C5 at (191.8, 31.9)
- removed the C5 at (56.8, 117.2)
- removed the C5 at (191.8, 117.2)
- removed the D1 at (170.5, 148.1)
- removed the D1 at (170.5, 62.8)
- removed the D1 at (35.5, 148.1)
- removed the D2 at (197.1, 83.9)
- removed the D2 at (62.1, 83.9)
- removed the D2 at (197.0, 169.2)
- removed the D2 at (62.0, 169.2)
- removed the D3 at (177.6, 52.9)
- removed the D3 at (42.6, 138.2)
- removed the D3 at (177.6, 138.2)
- removed the J1 at (83.3, 29.7)
- removed the J1 at (83.3, 115.0)
- removed the J1 at (218.3, 115.0)
- removed the J1 at (218.3, 29.7)
- removed the J2 at (158.6, 131.0)
- removed the J2 at (158.6, 45.6)
- removed the J2 at (23.6, 131.0)
- removed the J2 at (23.6, 45.6)
- removed the J3 at (266.1, 22.1)
- removed the J3 at (266.0, 107.4)
- removed the J3 at (131.1, 107.4)
- removed the J4 at (140.7, 63.5)
- removed the J4 at (140.7, 148.8)
- removed the J4 at (275.6, 148.8)
- removed the J4 at (275.6, 63.5)
- removed the J5 at (264.2, 89.4)
- removed the J5 at (264.2, 174.7)
- removed the J5 at (129.2, 174.7)
- removed the J5 at (129.3, 89.4)
- removed the J6 at (83.3, 21.1)
- removed the J6 at (218.2, 21.1)
- removed the J6 at (83.2, 106.4)
- removed the J6 at (218.2, 106.4)
- removed the J7 at (95.3, 106.4)
- removed the J7 at (230.3, 21.1)
- removed the J7 at (95.3, 21.1)
- removed the J7 at (230.3, 106.4)
- removed the J8 at (167.1, 129.3)
- removed the J8 at (32.2, 44.0)
- removed the J8 at (32.2, 129.3)
- removed the J8 at (167.2, 44.0)
- removed the R1 at (71.7, 81.5)
- removed the R1 at (206.7, 166.8)
- removed the R1 at (206.7, 81.5)
- removed the R1 at (71.7, 166.8)
- removed the R2 at (71.7, 83.6)
- removed the R2 at (206.7, 83.6)
- removed the R2 at (206.7, 168.9)
- removed the R2 at (71.7, 168.9)
- removed the R3 at (71.7, 170.9)
- removed the R3 at (206.7, 85.6)
- removed the R3 at (206.7, 170.9)
- removed the R3 at (71.7, 85.6)
- removed the R4 at (244.5, 83.2)
- removed the R4 at (109.5, 168.5)
- removed the R4 at (244.5, 168.5)
- removed the R5 at (170.2, 52.8)
- removed the R5 at (170.2, 138.1)
- removed the R5 at (35.2, 138.1)
- removed the R6 at (42.0, 148.3)
- removed the R6 at (177.0, 148.3)
- removed the R6 at (177.0, 63.0)
- removed the R7 at (265.2, 150.2)
- removed the R7 at (265.2, 64.9)
- removed the R7 at (130.2, 150.2)
- removed the R8 at (130.2, 153.2)
- removed the R8 at (265.2, 153.2)
- removed the R8 at (265.2, 67.8)
- removed the RN1 at (152.2, 16.7)
- removed the RN1 at (17.2, 102.0)
- removed the RN1 at (152.1, 102.0)
- removed the RN2 at (82.0, 124.0)
- removed the RN2 at (216.9, 124.0)
- removed the RN2 at (217.0, 38.6)
- removed the SW1 at (166.2, 36.8)
- removed the SW1 at (31.2, 122.2)
- removed the SW1 at (166.2, 122.2)
- removed the U1 at (232.6, 156.5)
- removed the U1 at (232.6, 71.2)
- removed the U1 at (97.6, 156.5)
- removed the U2 at (198.3, 56.2)
- removed the U2 at (198.3, 141.5)
- removed the U2 at (63.3, 141.5)
- removed the U3 at (184.2, 28.1)
- removed the U3 at (184.2, 113.4)
- removed the U3 at (49.2, 113.4)
- removed the U4 at (162.7, 84.9)
- removed the U4 at (27.7, 170.2)
- removed the U4 at (162.7, 170.2)
- added C7: 100nF, HomeBus:C_0805_2012Metric_Pad1.18x1.45mm_HandSolder, F.Cu at (64.8, 86.9)
- added C8: 100nF, HomeBus:C_0805_2012Metric_Pad1.18x1.45mm_HandSolder, F.Cu at (110.6, 80.7)
- added D2: WS2812B, LED_SMD:LED_WS2812B_PLCC4_5.0x5.0mm_P3.2mm, F.Cu at (70.5, 86.7)
- added D4: SMBJ26A, Diode_SMD:D_SMB, F.Cu at (32.5, 72.5)
- added D9: LED, LED_SMD:LED_1206_3216Metric_Pad1.42x1.75mm_HandSolder, F.Cu at (124.5, 87.0)
- added J1: IO Interface, HomeBus:PinSocket_1x10_P2.54mm_Vertical_SMD_Pin1Left, F.Cu at (94.2, 28.5)
- added J2: Conn_02x06_Odd_Even, Connector_PinSocket_2.54mm:PinSocket_2x06_P2.54mm_Vertical_SMD, F.Cu at (23.1, 55.8)
- added J4: I2C, HomeBus:PinSocket_1x04_P2.54mm_Vertical_SMD_Pin1Left, F.Cu at (139.0, 67.2)
- added J5: 24vdc, Connector_PinSocket_2.54mm:PinSocket_1x02_P2.54mm_Vertical_SMD_Pin1Left, F.Cu at (35.0, 44.8)
- added J6: Encoder 1, HomeBus:PinSocket_1x04_P2.54mm_Vertical_SMD_Pin1Left, F.Cu at (88.1, 19.4)
- added J7: Encoder 2, HomeBus:PinSocket_1x04_P2.54mm_Vertical_SMD_Pin1Left, F.Cu at (99.6, 19.5)
- added J8: WCH-LinkE Connector, HomeBus:IDC-Header_2x05_P2.54mm_Vertical_SMD, F.Cu at (135.2, 83.9)
- added R1: 330Ω, HomeBus:R_0805_2012Metric_Pad1.20x1.40mm_HandSolder, F.Cu at (77.8, 86.8)
- added R2: 10KΩ, HomeBus:R_0805_2012Metric_Pad1.20x1.40mm_HandSolder, F.Cu at (101.6, 84.2)
- added R3: 1kΩ, HomeBus:R_0805_2012Metric_Pad1.20x1.40mm_HandSolder, F.Cu at (124.9, 82.7)
- added SW2: RST, HomeBus:SW_SPST_PTS647_Sx38, F.Cu at (117.3, 89.9)
- added SW3: Boot, HomeBus:SW_SPST_PTS647_Sx38, F.Cu at (117.3, 83.7)
- C1, C2: footprint HomeBus:C_0603_1608Metric -> HomeBus:C_0805_2012Metric_Pad1.18x1.45mm_HandSolder
- C3, C5: footprint HomeBus:C_0603_1608Metric -> HomeBus:C_0805_2012Metric_Pad1.18x1.45mm_HandSolder; moved to B.Cu
- J3: footprint HomeBus:IDC-Header_2x10_P2.54mm_Horizontal -> Connector_PinSocket_2.54mm:PinSocket_2x10_P2.54mm_Vertical_SMD
- R4, R5, R6, R7, R8: footprint HomeBus:R_0805_2012Metric -> HomeBus:R_0805_2012Metric_Pad1.20x1.40mm_HandSolder
- moved J3 7.74 mm to (128.8, 29.5)
- moved R4 4.78 mm to (107.2, 79.0)
- moved C1 4.78 mm to (114.5, 71.4)
- moved C2 4.78 mm to (113.1, 69.9)
- moved U1 4.78 mm to (95.3, 67.0)
- moved C5 0.91 mm to (56.9, 30.9)
Connections:
- J3 pad 1: +5V -> GND
- J3 pad 10: Net-(J1-Pin_4) -> Net-(J1-Pin_3)
- J3 pad 11: Net-(J3-Pin_11) -> /SCL
- J3 pad 12: Net-(J3-Pin_12) -> /RX
- J3 pad 13: Net-(J3-Pin_13) -> Net-(J1-Pin_2)
- J3 pad 14: Net-(J3-Pin_14) -> /SDA
- J3 pad 15: Net-(J3-Pin_15) -> Net-(J1-Pin_5)
- J3 pad 16: Net-(J1-Pin_5) -> /RST
- J3 pad 17: Net-(J1-Pin_6) -> Net-(J3-Pin_18)
- J3 pad 18: Net-(J1-Pin_7) -> Net-(J3-Pin_17)
- J3 pad 19: Net-(J1-Pin_8) -> /SWCLK
- J3 pad 2: GND -> +5V
- J3 pad 20: Net-(J1-Pin_9) -> /SWDIO
- J3 pad 3: Net-(J3-Pin_3) -> Net-(J3-Pin_4)
- J3 pad 4: Net-(J3-Pin_4) -> Net-(J3-Pin_3)
- J3 pad 5: Net-(J3-Pin_5) -> Net-(J3-Pin_6)
- J3 pad 6: Net-(J3-Pin_6) -> Net-(J3-Pin_5)
- J3 pad 7: Net-(J1-Pin_1) -> /TX
- J3 pad 8: Net-(J1-Pin_2) -> Net-(J1-Pin_1)
- J3 pad 9: Net-(J1-Pin_3) -> Net-(J1-Pin_4)
- R4 pad 2: Net-(J3-Pin_15) -> /RST
- R7 pad 2: Net-(J1-Pin_7) -> /SDA
- R8 pad 2: Net-(J1-Pin_6) -> /SCL
- RN2 pad 6: Net-(J1-Pin_6) -> /SWDIO
- RN2 pad 7: Net-(J1-Pin_7) -> /SWCLK
- RN2 pad 8: Net-(J1-Pin_8) -> /RX
- RN2 pad 9: Net-(J1-Pin_9) -> /TX
- U1 pad 10: Net-(J3-Pin_11) -> /RX
- U1 pad 11: Net-(J3-Pin_13) -> /SDA
- U1 pad 12: Net-(J3-Pin_12) -> /SCL
- U1 pad 18: Net-(J1-Pin_9) -> /SWCLK
- U1 pad 20: Net-(J1-Pin_2) -> /TX
- U1 pad 3: Net-(J3-Pin_14) -> Net-(J1-Pin_2)
- U1 pad 4: Net-(J3-Pin_15) -> /RST
- U1 pad 5: Net-(J1-Pin_6) -> Net-(J3-Pin_17)
- U1 pad 6: Net-(J1-Pin_7) -> Net-(J3-Pin_18)
- U1 pad 8: Net-(J1-Pin_8) -> /SWDIO
- U3 pad 9: Net-(J3-Pin_14) -> Net-(J3-Pin_17)
- U4 pad 1: /+24vdc -> /+24V
Routing:
- net +5V: track 1402.9 -> 370.8 mm, vias 0 -> 3
- net Net-(J1-Pin_7): track 723.2 -> 0.00 mm, vias 4 -> 0
- net Net-(J1-Pin_6): track 694.5 -> 0.00 mm
- net Net-(J3-Pin_14): track 624.6 -> 0.00 mm, vias 4 -> 0
- net Net-(J3-Pin_11): track 515.6 -> 0.00 mm, vias 16 -> 0
- net Net-(J3-Pin_4): track 611.4 -> 146.5 mm, vias 8 -> 2
- net Net-(J1-Pin_4): track 600.8 -> 148.3 mm, vias 0 -> 5
- net Net-(J1-Pin_2): track 589.1 -> 154.4 mm, vias 0 -> 5
- net Net-(J3-Pin_12): track 410.8 -> 0.00 mm
- net Net-(J3-Pin_6): track 517.3 -> 120.4 mm, vias 0 -> 2
- net Net-(J3-Pin_3): track 514.2 -> 125.4 mm, vias 0 -> 2
- net Net-(J3-Pin_15): track 348.1 -> 0.00 mm
- net Net-(J3-Pin_13): track 345.1 -> 0.00 mm, vias 4 -> 0
- net Net-(J1-Pin_9): track 320.8 -> 0.00 mm
- net Net-(J1-Pin_8): track 319.4 -> 0.00 mm
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Other:
- board size 265 x 165.3 mm -> 130 x 80 mm
- board text added: "+12V"
- board text added: "Base Node Development Board V2.0"
- board text added: "GND"
- board text added: "HomeBus Base Node Devlopment Board V2.0 By:KV"
- board text added: "SW1"
- board text removed: "Base Node Test Board V2.0"
- board text removed: "RST"
- board text removed: "VCC"
